File: KiCad Files/keyboard.kicad_pcb (KiCad board)
At the start: 2 copper layers, 355.5 x 123 mm, 192 parts, among them J2 Button, J3 78171-0004, J5 Conn_01x03_Male, U1 SOT-23-5 5.5V 3.3V 500mA, U2 RP2040, Y1 3225_4P 12MHz

Commit message: routed matrix and updated git ignore
Parts:
- added C19: 10uf 0402, Capacitor_SMD:C_0402_1005Metric, B.Cu at (280.1, 60.0)
- moved J3 13.2 mm to (285.9, 46.1)
- moved R9 9.86 mm to (284.6, 54.3)
- moved F1 7.47 mm to (283.4, 51.6)
- moved D_49 3.15 mm to (77.7, 85.0)
- moved D_50 3.15 mm to (96.8, 85.0)
- moved D_51 3.15 mm to (115.8, 85.0)
- moved D_52 3.15 mm to (134.8, 85.0)
- moved D_53 3.15 mm to (153.9, 85.0)
- moved D_54 3.15 mm to (172.9, 85.0)
- moved D_55 3.15 mm to (192.0, 85.0)
- moved D_56 3.15 mm to (211.1, 85.0)
- moved D_57 3.15 mm to (230.1, 85.0)
- moved D_58 3.15 mm to (255.8, 85.0)
- moved C16 1.44 mm to (281.5, 66.4), turned to -135 degrees
- moved C5 1.20 mm to (281.4, 52.8)
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Connections:
- K_14 pad 1: col15 -> col14
- K_15 pad 1: col16 -> col15
- K_16 pad 1: col17 -> col16
- K_30 pad 1: col15 -> col14
- K_31 pad 1: col16 -> col15
- K_32 pad 1: col17 -> col16
- K_45 pad 1: col15 -> col14
- K_46 pad 1: col16 -> col15
- K_47 pad 1: col17 -> col16
- K_59 pad 1: col15 -> col14
- K_60 pad 1: col16 -> col15
- K_61 pad 1: col17 -> col16
- K_71 pad 1: col16 -> col15
- K_72 pad 1: col17 -> col16
- K_75 pad 1: col15 -> col14
- U2 pad 2: /GPIO0 -> col4
- U2 pad 27: /GPIO16 -> row3
- U2 pad 28: /GPIO17 -> row4
- U2 pad 29: /GPIO18 -> row0
- U2 pad 3: /GPIO1 -> col3
- U2 pad 30: /GPIO19 -> row1
- U2 pad 31: /GPIO20 -> row2
- U2 pad 32: /GPIO21 -> col13
- U2 pad 34: /GPIO22 -> col12
- U2 pad 35: /GPIO23 -> col11
- U2 pad 36: /GPIO24 -> col10
- U2 pad 37: /GPIO25 -> col9
- U2 pad 38: /GPIO26_ADC0 -> col8
- U2 pad 39: /GPIO27_ADC1 -> col7
- U2 pad 4: /GPIO2 -> col2
- U2 pad 40: /GPIO28_ADC2 -> col6
- U2 pad 41: /GPIO29_ADC3 -> col5
- U2 pad 5: /GPIO3 -> col1
- U2 pad 6: /GPIO4 -> col0
Routing:
- net row4: track 319.6 -> 627.5 mm
- net row0: track 335.8 -> 642.0 mm, vias 0 -> 2
- net col0: track 81.6 -> 379.8 mm
- net row1: track 343.8 -> 637.4 mm, vias 0 -> 4
- net row3: track 307.6 -> 591.6 mm
- net col1: track 84.5 -> 364.7 mm, vias 0 -> 1
- net col2: track 89.1 -> 361.2 mm
- net row2: track 375.5 -> 638.9 mm, vias 0 -> 4
- net col3: track 67.6 -> 319.4 mm
- net col4: track 87.7 -> 319.3 mm
- net col5: track 67.6 -> 280.1 mm
- net col6: track 87.1 -> 280.3 mm
- net col7: track 67.6 -> 241.6 mm
- net col8: track 90.3 -> 245.1 mm
- net col9: track 67.6 -> 203.2 mm
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
Commit message: added silkscreen markings, broke out unused GPIOs, cleaned up board, ran DRC and cleaned up traces.
Parts:
- added C1: 100nf 0402, Capacitor_SMD:C_0402_1005Metric, B.Cu at (318.1, 37.8)
- added C20: 100nf 0402, Capacitor_SMD:C_0402_1005Metric, B.Cu at (320.9, 37.0)
- added GTP1: GNDPAD, Connector_Wire:SolderWire-0.1sqmm_1x01_D0.4mm_OD1mm, F.Cu at (312.3, 73.9)
- added GTP2: GNDPAD, Connector_Wire:SolderWire-0.1sqmm_1x01_D0.4mm_OD1mm, F.Cu at (25.5, 72.7)
- added GTP3: GNDPAD, Connector_Wire:SolderWire-0.1sqmm_1x01_D0.4mm_OD1mm, F.Cu at (312.3, 93.0)
- added GTP4: GNDPAD, Connector_Wire:SolderWire-0.1sqmm_1x01_D0.4mm_OD1mm, F.Cu at (331.4, 35.8)
- added J1: Conn_01x10, Connector_PinHeader_1.00mm:PinHeader_1x10_P1.00mm_Vertical, F.Cu at (294.5, 68.5)
- added U3: TXS0101DCK, Package_TO_SOT_SMD:SOT-363_SC-70-6, B.Cu at (318.8, 35.8)
- moved D1 267.4 mm to (312.3, 35.8)
- moved D3 267.4 mm to (45.6, 54.9)
- moved D_16 16.6 mm to (332.6, 31.0)
- moved D_72 16.6 mm to (332.6, 107.2)
- moved D_32 16.6 mm to (332.6, 50.0)
- moved D_47 16.6 mm to (332.6, 69.1)
- moved D_61 16.6 mm to (332.6, 88.1)
- moved C17 0.72 mm to (293.0, 66.5), turned to -45 degrees
Connections:
- net 5V renamed VBUS
- C5 pad 1: VSYS -> +5V
- D1 pad 1: unconnected-(D1-VSS-Pad1) -> GND
- D1 pad 2: unconnected-(D1-DIN-Pad2) -> RGB_DATA_5V0
- D1 pad 3: unconnected-(D1-VDD-Pad3) -> +5V
- D2 pad 1: unconnected-(D2-VSS-Pad1) -> GND
- D2 pad 3: unconnected-(D2-VDD-Pad3) -> +5V
- D3 pad 1: unconnected-(D3-VSS-Pad1) -> GND
- D3 pad 3: unconnected-(D3-VDD-Pad3) -> +5V
- F1 pad 1: VSYS -> +5V
- U1 pad 1: VSYS -> +5V
- U2 pad 7: /GPIO5 -> RGB_DATA_3V3
Routing:
- net +5V: track 0.00 -> 389.3 mm, vias 0 -> 5
- net Net-(D1-DOUT): track 0.00 -> 224.1 mm, vias 0 -> 2
- net Net-(D2-DOUT): track 0.00 -> 134.8 mm, vias 0 -> 2
- net RGB_DATA_3V3: track 0.00 -> 64.2 mm
- net +3V3: track 42.2 -> 96.7 mm, vias 2 -> 3
- net GND: track 28.9 -> 50.2 mm, vias 22 -> 51
- net row3: track 591.6 -> 575.0 mm
- net row0: track 642.0 -> 625.4 mm
- net row4: track 627.5 -> 610.9 mm
- net row1: track 637.4 -> 622.5 mm
- net row2: track 638.9 -> 624.2 mm
- net /GPIO15: track 0.00 -> 12.8 mm
- net /GPIO14: track 0.00 -> 11.5 mm
- net /GPIO13: track 0.00 -> 10.4 mm
- net /GPIO12: track 0.00 -> 9.25 mm
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Other:
- board size 355.5 x 123 mm -> 333.4 x 100 mm
- board text added: "GND"
- board text added: "GP6 GP7 GP8 GP9 GP10 GP11 GP12 GP13 GP14 GP15"
- board text added: "SWC GND SWD"
- board text added: "env"
- board text added: "envious.design LASERman71 - Mini1800 V2 - Commission"

Commit message: added test points, cleaned up PCB, Generated production files
Parts:
- added TP1: TestPoint, TestPoint:TestPoint_Pad_D1.0mm, B.Cu at (277.2, 61.1)
- added TP2: TestPoint, TestPoint:TestPoint_Pad_D1.0mm, B.Cu at (282.2, 39.6)
- added TP3: TestPoint, TestPoint:TestPoint_Pad_D1.0mm, B.Cu at (280.2, 48.8)
- added TP4: TestPoint, TestPoint:TestPoint_Pad_D1.0mm, B.Cu at (326.1, 35.8)
- added TP5: TestPoint, TestPoint:TestPoint_Pad_D1.0mm, B.Cu at (323.7, 35.8)
- added TP6: TestPoint, TestPoint:TestPoint_Pad_D1.0mm, B.Cu at (289.8, 46.0)
- added TP7: TestPoint, TestPoint:TestPoint_Pad_D1.0mm, B.Cu at (285.5, 50.8)
- moved C9 0.98 mm to (284.6, 58.7)
Routing:
- net VBUS: track 8.00 -> 19.0 mm
- net RGB_DATA_3V3: track 64.2 -> 72.7 mm, vias 0 -> 2
- net RGB_DATA_5V0: track 6.29 -> 13.9 mm, vias 0 -> 2
- net GND: track 50.2 -> 57.6 mm
- net +5V: track 389.3 -> 392.9 mm
- net +1V1: track 13.1 -> 16.6 mm, vias 4 -> 5
- net +3V3: track 96.7 -> 100.1 mm
- net col15: track 78.7 -> 80.5 mm
- net D+: track 13.0 -> 14.8 mm
- net D-: track 13.0 -> 14.3 mm
Other:
- board text added: "3.3V"
- board text added: "3V3"
- board text added: "5V"
- board text added: "Bootsel"
- board text added: "RESET"
- board text added: "RGB DATA"
- board text added: "USB +D"
- board text added: "USB D-"
- board text added: "VBUS"
- board text added: "VSYS"
